Commit message: updated cmake

File: cartographer_ros/urdf/vlp32.urdf (robot description, URDF)
Before this commit: robot cartographer_backpack_3d, 3 links, 2 joints
Joints:
- joint sbg_link_joint: origin xyz=0 0 0 rpy=0 0 0 -> xyz=0 0 0 rpy=0 3.14159265359 0

Commit message: Further parameters for cartographer

File: cartographer_ros/urdf/vlp32.urdf (robot description, URDF)
Before this commit: robot cartographer_backpack_3d, 3 links, 2 joints
Joints:
- joint sbg_link_joint: origin xyz=0 0 0 rpy=0 3.14159265359 0 -> xyz=0 0 0 rpy=0 0 0
