Commit message: new tuning

File: cartographer_ros/urdf/pandar.urdf (robot description, URDF)
Before this commit: robot cartographer_backpack_3d, 3 links, 2 joints
Links:
- added link base_footprint; visual cylinder length=0.07 radius=0.05
- added link utm
Joints:
- added joint odom_link_joint: type fixed, parent utm, child base_footprint, origin xyz=0 0 0 rpy=0 0 0
- added joint oxts_link_joint: type fixed, parent base_link, child utm, origin xyz=1.90484 0 -0.699895 rpy=0 0 0
